File: 00-produccion-pcbs/1-versiones-profes/grupo-06/g-06-perc-02-rev-a/g-06-perc-02-rev-a.kicad_pcb (KiCad board)
At the start: 2 copper layers, 98.2 x 95.2 mm, 26 parts, among them J2 Barrel_Jack_Switch, J3 Barrel_Jack_Switch, J4 AudioJack2_SwitchT, SW3 SW_SPDT, U1 40106, U8 L7805, U9 4070

Commit message: añadido g06-02
Parts:
- added C7: 100n, Capacitor_THT:C_Disc_D5.0mm_W2.5mm_P2.50mm, F.Cu at (174.5, 83.5)
- C5: value 100u -> 100uF
- C6: value 10u -> 10uF
Connections:
- U1 pad 1: unconnected-(U1-Pad1) -> GND
- U1 pad 3: unconnected-(U1-Pad3) -> GND
- U9 pad 12: unconnected-(U9-Pad12) -> GND
- U9 pad 13: unconnected-(U9-Pad13) -> GND
Routing:
- net Net-(C4-Pad1): track 54.6 -> 56.0 mm
- net +5V: track 126.2 -> 127.4 mm
