File: 00-produccion-pcbs/1-versiones-profes/grupo-06/g-06-perc-02-rev-a/g-06-perc-02-rev-a.kicad_sch (KiCad schematic)
At the start: 27 parts, among them J2 Barrel_Jack_Switch, J3 Barrel_Jack_Switch, J4 AudioJack2_SwitchT, SW3 SW_SPDT, U1 40106, U8 L7805, U9 4070

Commit message: añadido g06-02
Connections:
- net GND: now also U1.1, U1.3, U9.12, U9.13
- no-connect marks 15 -> 11
